File: markmodel/markcircuit/markcircuit.kicad_sch (KiCad schematic)
At the start: 10 parts, among them J1 HC-05 (Bluetooth), J2 HW-493 (laser), J3 servo-motor_a, J4 servo-motor_b, J5 Barrel_Jack_MountingPin, U1 ATmega328-P, Y1 Crystal

Commit message: Schematic + symbols
Parts:
- removed C1: C, symbol Device:C
- removed J1: HC-05 (Bluetooth), symbol Connector:Conn_01x06_Socket
- removed J2: HW-493 (laser), symbol Connector:Conn_01x03_Pin
- removed J3: servo-motor_a, symbol Connector:Conn_01x03_Pin
- removed J4: servo-motor_b, symbol Connector:Conn_01x03_Pin
- removed J5: Barrel_Jack_MountingPin, symbol Connector:Barrel_Jack_MountingPin
- added C1: 22pF, symbol Device:C
- added C1: C, symbol Device:C
- added D1: LED, symbol Device:LED
- added HC-05: ~, symbol Mark_symbols:HC-05
- added HC-SR04: ~, symbol Mark_symbols:HC-SR04
- added LD1: D_Laser_1A3C, symbol Device:D_Laser_1A3C
- added M1, M2: Motor_Servo, symbol Motor:Motor_Servo
- added R2, R5: 220, symbol Device:R
- added R3: 10k, symbol Device:R
- added R3: 1k, symbol Device:R
- added R4: 2k, symbol Device:R
- added SW2: SW_DPST_x2, symbol Switch:SW_DPST_x2
- added SW3: SW_Push, symbol Switch:SW_Push
- C2: value C -> 22pF
- C3: value C -> 1uF
- XTAL1: renamed from Y1; value Crystal -> 16 MHz
Connections:
- net Reset: now reaches U1.1 (~{RESET}/PC6)
- net Reset: now also C3.1, R3.2, SW3.2
- net at U1.10 (XTAL2/PB7): now also C2.1, XTAL1.1
- net at U1.14 (PB0): now also HC-SR04.2 (ECHO)
- net at U1.15 (PB1): now also M1.1 (PWM)
- net at U1.16 (PB2): now also M2.1 (PWM)
- net at U1.17 (PB3): now also HC-SR04.3 (Trig)
- net Active_LED: now reaches U1.18 (PB4)
- net Active_LED: now also D1.2 (A)
- net at U1.2 (PD0): now also HC-05.3 (TXD)
- net 0: now reaches U1.22 (GND), U1.8 (GND)
- net 0: now also C2.2, C3.2, C1.1, C1.2, HC-05.4 (GND), HC-SR04.4 (GND), LD1.3 (K), M1.3 (-), M2.3 (-), R4.1, R5.2, SW3.1
- net at U1.3 (PD1): now also R3.1
- net at U1.5 (PD3): now also R2.1
- net at U1.7 (VCC): now also C1.2, SW2.1 (A)
- net at U1.9 (XTAL1/PB6): now also XTAL1.2, C1.1
- new net: LD1.1 (A), R2.2
- new net: D1.1 (K), R5.1
- new net: HC-05.2 (RXD), R3.2, R4.2
- new net Vcc: HC-05.5 (Vcc), HC-SR04.1 (Vcc), M1.2 (+), M2.2 (+), R3.1, SW2.2 (B)
- no-connect marks 0 -> 14
Other:
- moved on the sheet: XTAL1

Commit message: gabinete BIEN HECHO
Parts:
- C1: value C -> 10 uF
Changed lines of the file:
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@@
   )
   (symbol (lib_id "Device:C") (at 116.84 57.15 180) (unit 1)
-    (in_bom yes) (on_board yes) (dnp no) (fields_autoplaced)
+    (in_bom yes) (on_board yes) (dnp no)
     (property "Reference" "C1" (at 120.65 55.88 0)
       (effects (font (size 1.27 1.27)) (justify right))
     )
-    (property "Value" "C" (at 120.65 58.42 0)
+    (property "Value" "10 uF" (at 119.38 58.42 0)
       (effects (font (size 1.27 1.27)) (justify right))
     )

Commit message: finished.
Connections:
- net Active_LED: now also U1.14 (PB0); no longer U1.18 (PB4)
- net at R2.1: now also U1.6 (PD4); no longer U1.5 (PD3)
- net at HC-SR04.2 (ECHO): now also U1.5 (PD3); no longer U1.14 (PB0)
- net at HC-SR04.3 (Trig): now also U1.4 (PD2); no longer U1.17 (PB3)
Other:
- moved on the sheet: C1, C2, HC-05, HC-SR04, M1, M2, R2, R3, R4, XTAL1
